Commit message: Add inertia property

File: tutorial_robots/first_robot_description/urdf/common_properties.urdf.xacro (robot description, xacro)
@@ -9,3 +9,36 @@
         <color rgba="0 0 1 1"></color>
     </material>
+    <!-- macro for defining inertia for a box-->
+    <!-- Wiki page used to compute inertia values -->
+    <!-- https://en.wikipedia.org/wiki/List_of_moments_of_inertia#List_of_3D_inertia_tensors -->
+    <xacro:macro name="box_inertia" params="mass x y z origin_xyz origin_rpy">
+        <inertial>
+            <mass value="${mass}"></mass>
+            <origin xyz="${origin_xyz}" rpy="${origin_rpy}"></origin>
+            <inertia ixx="${(mass/12) * (y*y + z*z)}" ixy="0" ixz="0"
+                     iyy="${(mass/12) * (x*x + z*z)}" iyz="0"
+                     izz="${(mass/12) * (x*x + y*y)}">
+            </inertia>
+        </inertial>
+    </xacro:macro>
+    <xacro:macro name="cilinder_inertia" params="mass radius height origin_xyz origin_rpy">
+        <inertial>
+            <mass value="${mass}"></mass>
+            <origin xyz="${origin_xyz}" rpy="${origin_rpy}"></origin>
+            <inertia ixx="${(mass/12) * (3*radius*radius + height*height)}" ixy="0" ixz="0"
+                    iyy="${(mass/12) * (3*radius*radius + height*height)}" iyz="0"
+                    izz="${mass/2 * radius*radius}">
+            </inertia>
+        </inertial>
+    </xacro:macro>
+    <xacro:macro name="sphere_inertia" params="mass radius origin_xyz origin_rpy">
+        <inertial>
+            <mass value="${mass}"></mass>
+            <origin xyz="${origin_xyz}" rpy="${origin_rpy}"></origin>
+            <inertia ixx="${2/5*mass*radius*radius}" ixy="0" ixz="0"
+                    iyy="${2/5*mass*radius*radius}" iyz="0"
+                    izz="${2/5*mass*radius*radius}">
+            </inertia>
+        </inertial>
+    </xacro:macro>
 </robot>

File: tutorial_robots/first_robot_description/urdf/my_robot.urdf.xacro (robot description, xacro)
@@ -16,4 +16,7 @@
                 <material name="blue"></material>
             </visual>
+            <xacro:cilinder_inertia mass="1.0" radius="${radius}" height="${length}"
+                                    origin_xyz="0 0 0" origin_rpy="0 0 0">
+            </xacro:cilinder_inertia>
         </link>
     </xacro:macro>
@@ -31,8 +34,11 @@
             <material name="green"></material>
         </visual>
+        <xacro:box_inertia mass="5.0" x="${base_length}" y="${base_width}" z="${base_height}"
+                        origin_xyz="0 0 ${base_height/2.0}" origin_rpy="0 0 0">
+        </xacro:box_inertia>
     </link>
     <xacro:create_wheel prefix="right" radius="${wheel_radius}" length="${wheel_length}"></xacro:create_wheel>
     <xacro:create_wheel prefix="left" radius="${wheel_radius}" length="${wheel_length}"></xacro:create_wheel>
-        <link name="caster_wheel_link">
+    <link name="caster_wheel_link">
         <visual>
             <geometry>
@@ -41,4 +47,7 @@
             <origin xyz="0 0 0" rpy="0 0 0"></origin>
         </visual>
+        <xacro:sphere_inertia mass="0.5" radius="${wheel_radius/2.0}"
+                            origin_xyz="0 0 0" origin_rpy="0 0 0">
+        </xacro:sphere_inertia>
     </link>
     <!-- Joints -->
