Commit message: Update urdf to use xacro

File: tutorial_robots/first_robot_description/urdf/my_robot.urdf.xacro (robot description, xacro)
@@ -1,4 +1,9 @@
 <?xml version="1.0"?>
-<robot name="my_robot">
+<robot name="my_robot" xmlns:xacro="http://www.ros.org/wiki/xacro">
+    <xacro:property name="base_length" value="1.0"></xacro:property>
+    <xacro:property name="base_width" value="0.4"></xacro:property>
+    <xacro:property name="base_height" value="0.2"></xacro:property>
+    <xacro:property name="wheel_radius" value="0.1"></xacro:property>
+    <xacro:property name="wheel_length" value="0.05"></xacro:property>
     <material name="green">
         <!--red green blue alpha-->
@@ -13,5 +18,5 @@
         <parent link="world"></parent>
         <child link="base_link"></child>
-        <origin xyz="0 0 0.1" rpy="0 0 0"></origin>
+        <origin xyz="0 0 ${wheel_radius}" rpy="0 0 0"></origin>
     </joint>
     <link name="base_link">
@@ -19,9 +24,9 @@
             <geometry>
                 <!-- length, width, height-->
-                <box size="0.6 0.4 0.2"></box>
+                <box size="${base_length} ${base_width} ${base_height}"></box>
             </geometry>
             <!-- xyz = origin of the box-->
             <!-- rpy(rad) = roll(rotation on x) pitch(rotation on y) yaw(rotation on z)-->
-            <origin xyz="0 0 0.1" rpy="0 0 0"></origin>
+            <origin xyz="0 0 ${base_height/2.0}" rpy="0 0 0"></origin>
             <material name="green"></material>
         </visual>
@@ -30,7 +35,7 @@
         <visual>
             <geometry>
-                <cylinder radius="0.1" length="0.05"></cylinder>
+                <cylinder radius="${wheel_radius}" length="${wheel_length}"></cylinder>
             </geometry>
-            <origin xyz="0 0 0" rpy="1.57 0 0"></origin>
+            <origin xyz="0 0 0" rpy="${pi/2.0} 0 0"></origin>
             <material name="blue"></material>
         </visual>
@@ -39,5 +44,5 @@
         <parent link="base_link"></parent>
         <child link="right_wheel_link"></child>
-        <origin xyz="-0.15 -0.225 0" rpy="0 0 0"></origin>
+        <origin xyz="${-base_length/4} -${(base_width + wheel_length)/2.0} 0" rpy="0 0 0"></origin>
         <axis xyz="0 1 0"></axis>
     </joint>
@@ -45,14 +50,14 @@
         <visual>
             <geometry>
-                <cylinder radius="0.1" length="0.05"></cylinder>
+                <cylinder radius="${wheel_radius}" length="${wheel_length}"></cylinder>
             </geometry>
-            <origin xyz="0 0 0" rpy="1.57 0 0"></origin>
+            <origin xyz="0 0 0" rpy="${pi/2.0} 0 0"></origin>
             <material name="blue"></material>
         </visual>
     </link>
-    <joint name="left_right_wheel_joint" type="continuous">
+    <joint name="base_left_wheel_joint" type="continuous">
         <parent link="base_link"></parent>
         <child link="left_wheel_link"></child>
-        <origin xyz="-0.15 0.225 0" rpy="0 0 0"></origin>
+        <origin xyz="${-base_length/4} ${(base_width + wheel_length)/2.0} 0" rpy="0 0 0"></origin>
         <axis xyz="0 1 0"></axis>
     </joint>
@@ -60,5 +65,5 @@
         <visual>
             <geometry>
-                <sphere radius="0.05"></sphere>
+                <sphere radius="${wheel_radius/2.0}"></sphere>
             </geometry>
             <origin xyz="0 0 0" rpy="0 0 0"></origin>
@@ -68,5 +73,5 @@
         <parent link="base_link"></parent>
         <child link="caster_wheel_link"></child>
-        <origin xyz="0.2 0 -0.05" rpy="0 0 0"></origin>
+        <origin xyz="${base_length/3.0} 0 -${wheel_radius/2.0}" rpy="0 0 0"></origin>
         <limit lower="-3.14" upper="3.14" effort="100" velocity="100"></limit>
         <axis xyz="0 0 1" ></axis>

Commit message: Use macro to create the wheels

File: tutorial_robots/first_robot_description/urdf/my_robot.urdf.xacro (robot description, xacro)
@@ -4,6 +4,17 @@
     <xacro:property name="base_width" value="0.4"></xacro:property>
     <xacro:property name="base_height" value="0.2"></xacro:property>
-    <xacro:property name="wheel_radius" value="0.1"></xacro:property>
-    <xacro:property name="wheel_length" value="0.05"></xacro:property>
+    <xacro:property name="wheel_radius" value="0.2"></xacro:property>
+    <xacro:property name="wheel_length" value="0.1"></xacro:property>
+    <xacro:macro name="create_wheel" params="prefix radius length">
+        <link name="${prefix}_wheel_link">
+            <visual>
+                <geometry>
+                    <cylinder radius="${radius}" length="${length}"></cylinder>
+                </geometry>
+                <origin xyz="0 0 0" rpy="${pi/2.0} 0 0"></origin>
+                <material name="blue"></material>
+            </visual>
+        </link>
+    </xacro:macro>
     <material name="green">
         <!--red green blue alpha-->
@@ -14,10 +25,6 @@
         <color rgba="0 0 1 1"></color>
     </material>
+    <!-- Links -->
     <link name="world"></link>
-    <joint name="world_base_joint" type="fixed">
-        <parent link="world"></parent>
-        <child link="base_link"></child>
-        <origin xyz="0 0 ${wheel_radius}" rpy="0 0 0"></origin>
-    </joint>
     <link name="base_link">
         <visual>
@@ -32,35 +39,7 @@
         </visual>
     </link>
-    <link name="right_wheel_link">
-        <visual>
-            <geometry>
-                <cylinder radius="${wheel_radius}" length="${wheel_length}"></cylinder>
-            </geometry>
-            <origin xyz="0 0 0" rpy="${pi/2.0} 0 0"></origin>
-            <material name="blue"></material>
-        </visual>
-    </link>
-    <joint name="base_right_wheel_joint" type="continuous">
-        <parent link="base_link"></parent>
-        <child link="right_wheel_link"></child>
-        <origin xyz="${-base_length/4} -${(base_width + wheel_length)/2.0} 0" rpy="0 0 0"></origin>
-        <axis xyz="0 1 0"></axis>
-    </joint>
-    <link name="left_wheel_link">
-        <visual>
-            <geometry>
-                <cylinder radius="${wheel_radius}" length="${wheel_length}"></cylinder>
-            </geometry>
-            <origin xyz="0 0 0" rpy="${pi/2.0} 0 0"></origin>
-            <material name="blue"></material>
-        </visual>
-    </link>
-    <joint name="base_left_wheel_joint" type="continuous">
-        <parent link="base_link"></parent>
-        <child link="left_wheel_link"></child>
-        <origin xyz="${-base_length/4} ${(base_width + wheel_length)/2.0} 0" rpy="0 0 0"></origin>
-        <axis xyz="0 1 0"></axis>
-    </joint>
-    <link name="caster_wheel_link">
+    <xacro:create_wheel prefix="right" radius="${wheel_radius}" length="${wheel_length}"></xacro:create_wheel>
+    <xacro:create_wheel prefix="left" radius="${wheel_radius}" length="${wheel_length}"></xacro:create_wheel>
+        <link name="caster_wheel_link">
         <visual>
             <geometry>
@@ -70,4 +49,22 @@
         </visual>
     </link>
+    <!-- Joints -->
+    <joint name="world_base_joint" type="fixed">
+        <parent link="world"></parent>
+        <child link="base_link"></child>
+        <origin xyz="0 0 ${wheel_radius}" rpy="0 0 0"></origin>
+    </joint>
+    <joint name="base_right_wheel_joint" type="continuous">
+        <parent link="base_link"></parent>
+        <child link="right_wheel_link"></child>
+        <origin xyz="${-base_length/4} -${(base_width + wheel_length)/2.0} 0" rpy="0 0 0"></origin>
+        <axis xyz="0 1 0"></axis>
+    </joint>
+    <joint name="base_left_wheel_joint" type="continuous">
+        <parent link="base_link"></parent>
+        <child link="left_wheel_link"></child>
+        <origin xyz="${-base_length/4} ${(base_width + wheel_length)/2.0} 0" rpy="0 0 0"></origin>
+        <axis xyz="0 1 0"></axis>
+    </joint>
     <joint name="base_caster_wheel_joint" type="revolute">
         <parent link="base_link"></parent>

Commit message: Include xacro file from another xacro file

File: tutorial_robots/first_robot_description/urdf/my_robot.urdf.xacro (robot description, xacro)
@@ -1,4 +1,5 @@
 <?xml version="1.0"?>
 <robot name="my_robot" xmlns:xacro="http://www.ros.org/wiki/xacro">
+    <xacro:include filename="common_properties.urdf.xacro"></xacro:include>
     <xacro:property name="base_length" value="1.0"></xacro:property>
     <xacro:property name="base_width" value="0.4"></xacro:property>
@@ -17,12 +18,4 @@
         </link>
     </xacro:macro>
-    <material name="green">
-        <!--red green blue alpha-->
-        <color rgba="0 0.5 0 1"></color>
-    </material>
-    <material name="blue">
-        <!--red green blue alpha-->
-        <color rgba="0 0 1 1"></color>
-    </material>
     <!-- Links -->
     <link name="world"></link>

Commit message: Add collision property

File: tutorial_robots/first_robot_description/urdf/my_robot.urdf.xacro (robot description, xacro)
@@ -16,4 +16,12 @@
                 <material name="blue"></material>
             </visual>
+            <collision>
+                <!-- hack: for wheels collision is better to use a sphere(instead of cylinder)-->
+                <!-- shpere has only one point of collision -->
+                <geometry>
+                    <sphere radius="${wheel_radius}"></sphere>
+                </geometry>
+                <origin xyz="0 0 0" rpy="0 0 0"></origin>
+            </collision>
             <xacro:cilinder_inertia mass="1.0" radius="${radius}" height="${length}"
                                     origin_xyz="0 0 0" origin_rpy="0 0 0">
@@ -34,4 +42,10 @@
             <material name="green"></material>
         </visual>
+        <collision>
+            <geometry>
+                <box size="${base_length} ${base_width} ${base_height}"></box>
+            </geometry>
+            <origin xyz="0 0 ${base_height/2.0}" rpy="0 0 0"></origin>
+        </collision>
         <xacro:box_inertia mass="5.0" x="${base_length}" y="${base_width}" z="${base_height}"
                         origin_xyz="0 0 ${base_height/2.0}" origin_rpy="0 0 0">
@@ -47,4 +61,10 @@
             <origin xyz="0 0 0" rpy="0 0 0"></origin>
         </visual>
+        <collision>
+            <geometry>
+                <sphere radius="${wheel_radius/2.0}"></sphere>
+            </geometry>
+            <origin xyz="0 0 0" rpy="0 0 0"></origin>
+        </collision>
         <xacro:sphere_inertia mass="0.5" radius="${wheel_radius/2.0}"
                             origin_xyz="0 0 0" origin_rpy="0 0 0">

Commit message: Add gazebo plugins

File: tutorial_robots/first_robot_description/urdf/my_robot.urdf.xacro (robot description, xacro)
@@ -2,9 +2,10 @@
 <robot name="my_robot" xmlns:xacro="http://www.ros.org/wiki/xacro">
     <xacro:include filename="common_properties.urdf.xacro"></xacro:include>
+    <xacro:include filename="my_robot_gazebo.urdf.xacro"></xacro:include>
     <xacro:property name="base_length" value="1.0"></xacro:property>
     <xacro:property name="base_width" value="0.4"></xacro:property>
     <xacro:property name="base_height" value="0.2"></xacro:property>
-    <xacro:property name="wheel_radius" value="0.2"></xacro:property>
-    <xacro:property name="wheel_length" value="0.1"></xacro:property>
+    <xacro:property name="wheel_radius" value="0.1"></xacro:property>
+    <xacro:property name="wheel_length" value="0.05"></xacro:property>
     <xacro:macro name="create_wheel" params="prefix radius length">
         <link name="${prefix}_wheel_link">
@@ -89,10 +90,10 @@
         <axis xyz="0 1 0"></axis>
     </joint>
-    <joint name="base_caster_wheel_joint" type="revolute">
+    <joint name="base_caster_wheel_joint" type="fixed">
         <parent link="base_link"></parent>
         <child link="caster_wheel_link"></child>
         <origin xyz="${base_length/3.0} 0 -${wheel_radius/2.0}" rpy="0 0 0"></origin>
-        <limit lower="-3.14" upper="3.14" effort="100" velocity="100"></limit>
-        <axis xyz="0 0 1" ></axis>
+        <!-- <limit lower="-3.14" upper="3.14" effort="100" velocity="100"></limit> -->
+        <!-- <axis xyz="0 0 1" ></axis> -->
     </joint>
 </robot>
