Commit message: Use different urdf

File: tutorial_robots/first_robot_description/urdf/mobile_base_gazebo.xacro (robot description, xacro)
@@ -2,6 +2,6 @@
 <robot xmlns:xacro="http://www.ros.org/wiki/xacro">
     <gazebo reference="caster_wheel_link">
-        <mu1 value="0.1"></mu1>
-        <mu2 value="0.1"></mu2>
+        <mu1 value="0.1" />
+        <mu2 value="0.1" />
     </gazebo>
     <gazebo>
@@ -14,5 +14,5 @@
             <wheel_radius>0.1</wheel_radius>
             <frame_id>odom</frame_id>
-            <child_frame_id>world</child_frame_id>
+            <child_frame_id>base_footprint</child_frame_id>
         </plugin>
     </gazebo>

File: tutorial_robots/first_robot_description/urdf/my_robot.urdf.xacro (robot description, xacro)
@@ -1,99 +1,6 @@
 <?xml version="1.0"?>
 <robot name="my_robot" xmlns:xacro="http://www.ros.org/wiki/xacro">
-    <xacro:include filename="common_properties.urdf.xacro"></xacro:include>
-    <xacro:include filename="my_robot_gazebo.urdf.xacro"></xacro:include>
-    <xacro:property name="base_length" value="1.0"></xacro:property>
-    <xacro:property name="base_width" value="0.4"></xacro:property>
-    <xacro:property name="base_height" value="0.2"></xacro:property>
-    <xacro:property name="wheel_radius" value="0.1"></xacro:property>
-    <xacro:property name="wheel_length" value="0.05"></xacro:property>
-    <xacro:macro name="create_wheel" params="prefix radius length">
-        <link name="${prefix}_wheel_link">
-            <visual>
-                <geometry>
-                    <cylinder radius="${radius}" length="${length}"></cylinder>
-                </geometry>
-                <origin xyz="0 0 0" rpy="${pi/2.0} 0 0"></origin>
-                <material name="blue"></material>
-            </visual>
-            <collision>
-                <!-- hack-for wheels collision is better to use a sphere(instead of cylinder)-->
-                <!-- shpere has only one point of collision -->
-                <geometry>
-                    <sphere radius="${wheel_radius}"></sphere>
-                </geometry>
-                <origin xyz="0 0 0" rpy="0 0 0"></origin>
-            </collision>
-            <xacro:cilinder_inertia mass="1.0" radius="${radius}" height="${length}"
-                                    origin_xyz="0 0 0" origin_rpy="0 0 0">
-            </xacro:cilinder_inertia>
-        </link>
-    </xacro:macro>
-    <!-- Links -->
-    <link name="world"></link>
-    <link name="base_link">
-        <visual>
-            <geometry>
-                <!-- length, width, height-->
-                <box size="${base_length} ${base_width} ${base_height}"></box>
-            </geometry>
-            <!-- xyz = origin of the box-->
-            <!-- rpy(rad) = roll(rotation on x) pitch(rotation on y) yaw(rotation on z)-->
-            <origin xyz="0 0 ${base_height/2.0}" rpy="0 0 0"></origin>
-            <material name="green"></material>
-        </visual>
-        <collision>
-            <geometry>
-                <box size="${base_length} ${base_width} ${base_height}"></box>
-            </geometry>
-            <origin xyz="0 0 ${base_height/2.0}" rpy="0 0 0"></origin>
-        </collision>
-        <xacro:box_inertia mass="5.0" x="${base_length}" y="${base_width}" z="${base_height}"
-                        origin_xyz="0 0 ${base_height/2.0}" origin_rpy="0 0 0">
-        </xacro:box_inertia>
-    </link>
-    <xacro:create_wheel prefix="right" radius="${wheel_radius}" length="${wheel_length}"></xacro:create_wheel>
-    <xacro:create_wheel prefix="left" radius="${wheel_radius}" length="${wheel_length}"></xacro:create_wheel>
-    <link name="caster_wheel_link">
-        <visual>
-            <geometry>
-                <sphere radius="${wheel_radius/2.0}"></sphere>
-            </geometry>
-            <origin xyz="0 0 0" rpy="0 0 0"></origin>
-        </visual>
-        <collision>
-            <geometry>
-                <sphere radius="${wheel_radius/2.0}"></sphere>
-            </geometry>
-            <origin xyz="0 0 0" rpy="0 0 0"></origin>
-        </collision>
-        <xacro:sphere_inertia mass="0.5" radius="${wheel_radius/2.0}"
-                            origin_xyz="0 0 0" origin_rpy="0 0 0">
-        </xacro:sphere_inertia>
-    </link>
-    <!-- Joints -->
-    <joint name="world_base_joint" type="fixed">
-        <parent link="world"></parent>
-        <child link="base_link"></child>
-        <origin xyz="0 0 ${wheel_radius}" rpy="0 0 0"></origin>
-    </joint>
-    <joint name="base_right_wheel_joint" type="continuous">
-        <parent link="base_link"></parent>
-        <child link="right_wheel_link"></child>
-        <origin xyz="${-base_length/4} -${(base_width + wheel_length)/2.0} 0" rpy="0 0 0"></origin>
-        <axis xyz="0 1 0"></axis>
-    </joint>
-    <joint name="base_left_wheel_joint" type="continuous">
-        <parent link="base_link"></parent>
-        <child link="left_wheel_link"></child>
-        <origin xyz="${-base_length/4} ${(base_width + wheel_length)/2.0} 0" rpy="0 0 0"></origin>
-        <axis xyz="0 1 0"></axis>
-    </joint>
-    <joint name="base_caster_wheel_joint" type="fixed">
-        <parent link="base_link"></parent>
-        <child link="caster_wheel_link"></child>
-        <origin xyz="${base_length/3.0} 0 -${wheel_radius/2.0}" rpy="0 0 0"></origin>
-        <!-- <limit lower="-3.14" upper="3.14" effort="100" velocity="100"></limit> -->
-        <!-- <axis xyz="0 0 1" ></axis> -->
-    </joint>
+    <xacro:include filename="common_properties.xacro" />
+    <xacro:include filename="mobile_base.xacro" />
+    <xacro:include filename="mobile_base_gazebo.xacro" />
 </robot>

File: tutorial_robots/first_robot_description/urdf_/common_properties.urdf.xacro (robot description, xacro)
@@ -32,5 +32,5 @@
         </inertial>
     </xacro:macro>
-    <xacro:macro name="sphere_inertia" params="mass radius origin_xyz origin_rpy">
+    <!-- <xacro:macro name="sphere_inertia" params="mass radius origin_xyz origin_rpy">
         <inertial>
             <mass value="${mass}"></mass>
@@ -41,4 +41,34 @@
             </inertia>
         </inertial>
+    </xacro:macro> -->
+    <material name="grey">
+        <color rgba="0.5 0.5 0.5 1" />
+    </material>
+    <!-- <xacro:macro name="box_inertia" params="m x y z o_xyz o_rpy">
+        <inertial>
+            <mass value="${m}" />
+            <origin xyz="${o_xyz}" rpy="${o_rpy}" />
+            <inertia ixx="${(m/12) * (y*y + z*z)}" ixy="0" ixz="0"
+                     iyy="${(m/12) * (x*x + z*z)}" iyz="0"
+                     izz="${(m/12) * (x*x + y*y)}" />
+        </inertial>
+    </xacro:macro> -->
+    <xacro:macro name="cylinder_inertia" params="m r l o_xyz o_rpy">
+        <inertial>
+            <mass value="${m}" />
+            <origin xyz="${o_xyz}" rpy="${o_rpy}" />
+            <inertia ixx="${(m/12) * (3*r*r + l*l)}" ixy="0" ixz="0"
+                     iyy="${(m/12) * (3*r*r + l*l)}" iyz="0"
+                     izz="${(m/2) * (r*r)}" />
+        </inertial>
+    </xacro:macro>
+    <xacro:macro name="sphere_inertia" params="m r o_xyz o_rpy">
+        <inertial>
+            <mass value="${m}" />
+            <origin xyz="${o_xyz}" rpy="${o_rpy}" />
+            <inertia ixx="${(2/5) * m * r * r}" ixy="0" ixz="0"
+                     iyy="${(2/5) * m * r * r}" iyz="0"
+                     izz="${(2/5) * m * r * r}" />
+        </inertial>
     </xacro:macro>
 </robot>
