Commit message: Add 2 segment arm to existing robot

File: tutorial_robots/first_robot_description/urdf/common_properties.xacro (robot description, xacro)
@@ -6,4 +6,7 @@
     <material name="grey">
         <color rgba="0.5 0.5 0.5 1" />
+    </material>
+    <material name="orange">
+        <color rgba="0.9 0.3 0.01 1"></color>
     </material>
     <xacro:macro name="box_inertia" params="m x y z o_xyz o_rpy">

File: tutorial_robots/first_robot_description/urdf/my_robot.urdf.xacro (robot description, xacro)
@@ -5,3 +5,4 @@
     <xacro:include filename="mobile_base_gazebo.xacro" />
     <xacro:include filename="camera.xacro" />
+    <xacro:include filename="arm.xacro"/>
 </robot>
