Commit message: Complete robot arm

File: tutorial_robots/first_robot_description/urdf/arm.xacro (robot description, xacro)
@@ -4,5 +4,5 @@
     <xacro:property name="arm_base_width" value="0.1"></xacro:property>
     <xacro:property name="arm_base_height" value="0.02"></xacro:property>
-    <xacro:property name="arm_base_mass" value="0.1"></xacro:property>
+    <xacro:property name="arm_base_mass" value="0.5"></xacro:property>
     <xacro:property name="forearm_radius" value="0.02"></xacro:property>
     <xacro:property name="forearm_length" value="0.3"></xacro:property>
@@ -16,5 +16,5 @@
                 <box size="${arm_base_length} ${arm_base_width} ${arm_base_height}"></box>
             </geometry>
-            <origin xyz="0 0 0" rpy="0 0 0"></origin>
+            <origin xyz="0 0 ${arm_base_height/2}" rpy="0 0 0"></origin>
             <material name="orange"></material>
         </visual>
@@ -23,8 +23,8 @@
                 <box size="${arm_base_length} ${arm_base_width} ${arm_base_height}"></box>
             </geometry>
-            <origin xyz="0 0 0" rpy="0 0 0"></origin>
+            <origin xyz="0 0 ${arm_base_height/2}" rpy="0 0 0"></origin>
         </collision>
         <xacro:box_inertia m="${arm_base_mass}" x="${arm_base_length}" y="${arm_base_width}" z="${arm_base_height}"
-                            o_xyz="0 0 ${base_height}" o_rpy="0 0 0"></xacro:box_inertia>
+                            o_xyz="0 0 ${arm_base_height/2}" o_rpy="0 0 0"></xacro:box_inertia>
     </link>
     <link name="forearm_link">
@@ -43,5 +43,5 @@
         </collision>
         <xacro:cylinder_inertia m="${forearm_mass}" r="${forearm_radius}" l="${forearm_length}"
-                                o_xyz="0 0 0" o_rpy="0 0 0"></xacro:cylinder_inertia>
+                                o_xyz="0 0 ${forearm_length/2}" o_rpy="0 0 0"></xacro:cylinder_inertia>
     </link>
     <link name="hand_link">
@@ -59,17 +59,18 @@
         </collision>
         <xacro:cylinder_inertia m="${hand_mass}" r="${hand_radius}" l="${hand_length}"
-                                o_xyz="0 0 0" o_rpy="0 0 0"></xacro:cylinder_inertia>
+                                o_xyz="0 0 ${hand_length/2}" o_rpy="0 0 0"></xacro:cylinder_inertia>
     </link>
     <joint name="arm_base_joint" type="fixed">
         <parent link="base_link"></parent>
         <child link="arm_base_link"></child>
-        <origin xyz="0 0 ${base_height + arm_base_height/2}" rpy="0 0 0"></origin>
+        <origin xyz="0 0 ${base_height}" rpy="0 0 0"></origin>
     </joint>
     <joint name="arm_base_forearm_joint" type="revolute">
         <parent link="arm_base_link"></parent>
         <child link="forearm_link"></child>
-        <origin xyz="0 0 0" rpy="0 0 0"></origin>
+        <origin xyz="0 0 ${arm_base_height}" rpy="0 0 0"></origin>
         <axis xyz="0 1 0"></axis>
         <limit lower="0.0" upper="${pi/2.0}" effort="10" velocity="10"></limit>
+        <dynamics friction="0.3" damping="0.3"></dynamics>
     </joint>
     <joint name="forearm_hand_joint" type="revolute">
@@ -79,4 +80,5 @@
         <axis xyz="0 1 0"></axis>
         <limit lower="0.0" upper="${pi/2.0}" effort="10" velocity="10"></limit>
+        <dynamics friction="0.3" damping="0.3"></dynamics>
     </joint>
 </robot>

File: tutorial_robots/first_robot_description/urdf/my_robot.urdf.xacro (robot description, xacro)
@@ -6,3 +6,4 @@
     <xacro:include filename="camera.xacro" />
     <xacro:include filename="arm.xacro"/>
+    <xacro:include filename="arm_gazebo.xacro"/>
 </robot>
