Commit message: Create moveit config package

File: tutorial_robots/robot_arm_description/urdf/links_macro.xacro (robot description, xacro)
@@ -10,4 +10,10 @@
                 <material name="${material}"></material>
             </visual>
+            <collision>
+                <geometry>
+                    <box size="${length} ${width} ${height}"></box>
+                </geometry>
+                <origin xyz="${origin_xyz}" rpy="0 0 0"></origin>
+            </collision>
         </link>
     </xacro:macro>
@@ -21,4 +27,11 @@
                 <material name="${material}"></material>
             </visual>
+            <!-- use box instead of cylinder for simpler collision computations -->
+            <collision>
+                <geometry>
+                    <box size="${radius*2.0} ${radius*2.0} ${length}"></box>
+                </geometry>
+                <origin xyz="${origin_xyz}" rpy="0 0 0"></origin>
+            </collision>
         </link>
     </xacro:macro>
