Commit message: Finish implementation for robot arm description

File: tutorial_robots/robot_arm_description/urdf/arm.xacro (robot description, xacro)
@@ -1,4 +1,4 @@
 <?xml version="1.0"?>
-<robot name="robot_arm" xmlns:xacro="http://www.ros.org/wiki/xacro">
+<robot xmlns:xacro="http://www.ros.org/wiki/xacro">
     <xacro:include filename="colors.xacro"></xacro:include>
     <xacro:include filename="links_macro.xacro"></xacro:include>
@@ -6,13 +6,6 @@
     <xacro:property name="base_link_width" value="0.5"></xacro:property>
     <xacro:property name="base_link_height" value="0.2"></xacro:property>
-    <link name="base_link">
-        <visual>
-            <geometry>
-                <box size="${base_link_length} ${base_link_width} ${base_link_height}"></box>
-            </geometry>
-            <origin xyz="0 0 ${base_link_height/2.0}" rpy="0 0 0"></origin>
-            <material name="grey"></material>
-        </visual>
-    </link>
+    <xacro:box_link name="base_link" length="${base_link_length}" width="${base_link_width}" height="${base_link_height}"
+                    origin_xyz="0 0 ${base_link_height/2.0}" material="grey"></xacro:box_link>
     <xacro:property name="shoulder_link_length" value="0.5"></xacro:property>
     <xacro:property name="shoulder_link_radius" value="0.1"></xacro:property>
@@ -31,4 +24,15 @@
     <xacro:cylinder_link name="foream_link" length="${forearm_link_length}" radius="${forearm_link_radius}"
                             origin_xyz="0 0 ${forearm_link_length/2.0}" material="grey"></xacro:cylinder_link>
+    <xacro:property name="wrist_link_length" value="0.1"></xacro:property>
+    <xacro:property name="wrist_link_width" value="0.1"></xacro:property>
+    <xacro:property name="wrist_link_height" value="0.05"></xacro:property>
+    <xacro:box_link name="wrist_link" length="${wrist_link_length}" width="${wrist_link_width}" height="${wrist_link_height}"
+                    origin_xyz="0 0 ${wrist_link_height/2.0}" material="blue"></xacro:box_link>
+    <xacro:property name="hand_link_length" value="0.1"></xacro:property>
+    <xacro:property name="hand_link_width" value="0.1"></xacro:property>
+    <xacro:property name="hand_link_height" value="0.02"></xacro:property>
+    <xacro:box_link name="hand_link" length="${hand_link_length}" width="${hand_link_width}" height="${hand_link_height}"
+                    origin_xyz="0 0 ${hand_link_height/2.0}" material="grey"></xacro:box_link>
+    <link name="tool_link"></link>
     <!-- Joints -->
     <!-- 1 -->
@@ -64,3 +68,24 @@
         <limit effort="100.0" velocity="1.0" lower="-3.14" upper="3.14"></limit>
     </joint>
+    <!-- 5 -->
+    <joint name="forearm_wrist_joint" type="revolute">
+        <parent link="foream_link"></parent>
+        <child link="wrist_link"></child>
+        <origin xyz="0 0 ${forearm_link_length}" rpy="0 0 0"></origin>
+        <axis xyz="0 1 0"></axis>
+        <limit effort="100.0" velocity="1.0" lower="-1.57" upper="1.57"></limit>
+    </joint>
+    <!-- 6 -->
+    <joint name="wrist_hand_joint" type="continuous">
+        <parent link="wrist_link"></parent>
+        <child link="hand_link"></child>
+        <origin xyz="0 0 ${wrist_link_height}" rpy="0 0 0"></origin>
+        <axis xyz="0 0 1"></axis>
+    </joint>
+    <!-- 7 -->
+    <joint name="hand_tool_joint" type="fixed">
+        <parent link="hand_link"></parent>
+        <child link="tool_link"></child>
+        <origin xyz="0 0 ${hand_link_height}"></origin>
+    </joint>
 </robot>

File: tutorial_robots/robot_arm_description/urdf/links_macro.xacro (robot description, xacro)
@@ -1,6 +1,6 @@
 <?xml version="1.0"?>
 <robot xmlns:xacro="http://www.ros.org/wiki/xacro">
-    <xacro:macro name="box_link" params="length width height origin_xyz material">
-        <link name="base_link">
+    <xacro:macro name="box_link" params="name length width height origin_xyz material">
+        <link name="${name}">
             <visual>
                 <geometry>
@@ -8,5 +8,5 @@
                 </geometry>
                 <origin xyz="${origin_xyz}" rpy="0 0 0"></origin>
-                <material name="material"></material>
+                <material name="${material}"></material>
             </visual>
         </link>

Commit message: Fix review findings

File: tutorial_robots/robot_arm_description/urdf/arm.xacro (robot description, xacro)
@@ -22,5 +22,5 @@
     <xacro:property name="forearm_link_length" value="0.5"></xacro:property>
     <xacro:property name="forearm_link_radius" value="0.05"></xacro:property>
-    <xacro:cylinder_link name="foream_link" length="${forearm_link_length}" radius="${forearm_link_radius}"
+    <xacro:cylinder_link name="forearm_link" length="${forearm_link_length}" radius="${forearm_link_radius}"
                             origin_xyz="0 0 ${forearm_link_length/2.0}" material="grey"></xacro:cylinder_link>
     <xacro:property name="wrist_link_length" value="0.1"></xacro:property>
@@ -63,5 +63,5 @@
     <joint name="elbow_forearm_joint" type="revolute">
         <parent link="elbow_link"></parent>
-        <child link="foream_link"></child>
+        <child link="forearm_link"></child>
         <origin xyz="0 0 ${elbow_link_length}" rpy="0 0 0"></origin>
         <axis xyz="0 0 1"></axis>
@@ -70,5 +70,5 @@
     <!-- 5 -->
     <joint name="forearm_wrist_joint" type="revolute">
-        <parent link="foream_link"></parent>
+        <parent link="forearm_link"></parent>
         <child link="wrist_link"></child>
         <origin xyz="0 0 ${forearm_link_length}" rpy="0 0 0"></origin>

Commit message: Add gripper to robot arm

File: tutorial_robots/robot_arm_description/urdf/arm.xacro (robot description, xacro)
@@ -1,6 +1,4 @@
 <?xml version="1.0"?>
 <robot xmlns:xacro="http://www.ros.org/wiki/xacro">
-    <xacro:include filename="colors.xacro"></xacro:include>
-    <xacro:include filename="links_macro.xacro"></xacro:include>
     <xacro:property name="base_link_length" value="0.5"></xacro:property>
     <xacro:property name="base_link_width" value="0.5"></xacro:property>

File: tutorial_robots/robot_arm_description/urdf/colors.xacro (robot description, xacro)
@@ -7,3 +7,9 @@
         <color rgba="0 0 0.5 1"></color>
     </material>
+    <material name="dark_green">
+        <color rgba="0 0.4 0 1"></color>
+    </material>
+    <material name="light_green">
+        <color rgba="0 0.6 0 1"></color>
+    </material>
 </robot>

File: tutorial_robots/robot_arm_description/urdf/robot_arm.xacro (robot description, xacro)
@@ -1,4 +1,13 @@
 <?xml version="1.0"?>
 <robot name="robot_arm" xmlns:xacro="http://www.ros.org/wiki/xacro">
+    <xacro:include filename="colors.xacro"></xacro:include>
+    <xacro:include filename="links_macro.xacro"></xacro:include>
     <xacro:include filename="arm.xacro"></xacro:include>
+    <xacro:include filename="gripper.xacro"></xacro:include>
+    <!-- 8 -->
+    <joint name="tool_gripper_joint" type="fixed">
+        <parent link="tool_link"></parent>
+        <child link="gripper_base_link"></child>
+        <origin xyz="0 0 0" rpy="0 0 0"></origin>
+    </joint>
 </robot>

Commit message: Create ros action server to interact with robot arm

File: tutorial_robots/robot_arm_description/urdf/arm.xacro (robot description, xacro)
@@ -80,4 +80,5 @@
         <origin xyz="0 0 ${wrist_link_height}" rpy="0 0 0"></origin>
         <axis xyz="0 0 1"></axis>
+        <limit effort="100.0" velocity="1.0"/>
     </joint>
     <!-- 7 -->

File: tutorial_robots/robot_arm_description/urdf/robot_arm.ros2_control.xacro (robot description, xacro)
@@ -48,4 +48,11 @@
           </state_interface>
       </joint>
+      <joint name="gripper_right_finger_joint">
+          <param name="mimic">gripper_left_finger_joint</param>
+          <param name="multiplier">-1.0</param>
+          <state_interface name="position">
+            <param name="initial_value">0</param>
+          </state_interface>
+      </joint>
   </ros2_control>
 </robot>

Commit message: Update robot arm - add inertia to links - add new object to robot world - define extra robot arm positions

File: tutorial_robots/robot_arm_description/urdf/arm.xacro (robot description, xacro)
@@ -1,4 +1,5 @@
 <?xml version="1.0"?>
 <robot xmlns:xacro="http://www.ros.org/wiki/xacro">
+    <link name="base_footprint"></link>
     <xacro:property name="base_link_length" value="0.5"></xacro:property>
     <xacro:property name="base_link_width" value="0.5"></xacro:property>
@@ -32,6 +33,19 @@
     <xacro:box_link name="hand_link" length="${hand_link_length}" width="${hand_link_width}" height="${hand_link_height}"
                     origin_xyz="0 0 ${hand_link_height/2.0}" material="grey"></xacro:box_link>
-    <link name="tool_link"></link>
+    <link name="tool_link">
+        <inertial>
+            <origin xyz="0 0 0" rpy="0 0 0"></origin>
+            <mass value="0.001"></mass>
+            <inertia ixx="1e-6" ixy="0.0" ixz="0.0" iyy="1e-6" iyz="0.0" izz="1e-6"></inertia>
+        </inertial>
+    </link>
     <!-- Joints -->
+    <!-- Virtual joint to connect the robot to the world frame -->
+    <joint name="base_footprint_joint" type="fixed">
+        <parent link="base_footprint"></parent>
+        <child link="base_link"></child>
+        <origin xyz="0 0 0" rpy="0 0 0"></origin>
+        <dynamics friction="0.5" damping="0.5"/>
+    </joint>
     <!-- 1 -->
     <joint name="base_shoulder_joint" type="revolute">
@@ -41,4 +55,5 @@
         <axis xyz="0 0 1"></axis>
         <limit effort="100.0" velocity="1.0" lower="-3.14" upper="3.14"></limit>
+        <dynamics friction="0.5" damping="0.5"/>
     </joint>
     <!-- 2 -->
@@ -49,4 +64,5 @@
         <axis xyz="0 1 0"></axis>
         <limit effort="100.0" velocity="1.0" lower="0.0" upper="2.5"></limit>
+        <dynamics friction="0.5" damping="0.5"/>
     </joint>
     <!-- 3 -->
@@ -57,4 +73,5 @@
         <axis xyz="0 1 0"></axis>
         <limit effort="100.0" velocity="1.0" lower="0.0" upper="2.5"></limit>
+        <dynamics friction="0.5" damping="0.5"/>
     </joint>
     <!-- 4 -->
@@ -65,4 +82,5 @@
         <axis xyz="0 0 1"></axis>
         <limit effort="100.0" velocity="1.0" lower="-3.14" upper="3.14"></limit>
+        <dynamics friction="0.5" damping="0.5"/>
     </joint>
     <!-- 5 -->
@@ -73,4 +91,5 @@
         <axis xyz="0 1 0"></axis>
         <limit effort="100.0" velocity="1.0" lower="-1.57" upper="1.57"></limit>
+        <dynamics friction="0.5" damping="0.5"/>
     </joint>
     <!-- 6 -->

File: tutorial_robots/robot_arm_description/urdf/gripper.xacro (robot description, xacro)
@@ -25,5 +25,4 @@
         <origin xyz="${gripper_base_link_length/2.0} 0 ${gripper_base_link_height}" rpy="0 0 0"></origin>
         <axis xyz="1 0 0 "></axis>
-        <mimic joint="gripper_left_finger_joint" multiplier="-1.0"></mimic>
         <limit effort="100.0" velocity="1.0" lower="-${0.1 - finger_link_width/3.0}" upper="0.0"></limit>
     </joint>

File: tutorial_robots/robot_arm_description/urdf/links_macro.xacro (robot description, xacro)
@@ -1,5 +1,10 @@
 <?xml version="1.0"?>
 <robot xmlns:xacro="http://www.ros.org/wiki/xacro">
+    <xacro:property name="default_density" value="500.0"></xacro:property>
     <xacro:macro name="box_link" params="name length width height origin_xyz material">
+        <xacro:property name="mass" value="${default_density * length * width * height}"></xacro:property>
+        <xacro:property name="ixx" value="${mass * (width*width + height*height) / 12.0}"></xacro:property>
+        <xacro:property name="iyy" value="${mass * (length*length + height*height) / 12.0}"></xacro:property>
+        <xacro:property name="izz" value="${mass * (length*length + width*width) / 12.0}"></xacro:property>
         <link name="${name}">
             <visual>
@@ -16,7 +21,16 @@
                 <origin xyz="${origin_xyz}" rpy="0 0 0"></origin>
             </collision>
+            <inertial>
+                <origin xyz="${origin_xyz}" rpy="0 0 0"></origin>
+                <mass value="${mass}"></mass>
+                <inertia ixx="${ixx}" ixy="0.0" ixz="0.0" iyy="${iyy}" iyz="0.0" izz="${izz}"></inertia>
+            </inertial>
         </link>
     </xacro:macro>
     <xacro:macro name="cylinder_link" params="name length radius origin_xyz material">
+        <xacro:property name="mass" value="${default_density * 3.14159265359 * radius * radius * length}"></xacro:property>
+        <xacro:property name="ixx" value="${mass * (3.0*radius*radius + length*length) / 12.0}"></xacro:property>
+        <xacro:property name="iyy" value="${mass * (3.0*radius*radius + length*length) / 12.0}"></xacro:property>
+        <xacro:property name="izz" value="${mass * radius * radius / 2.0}"></xacro:property>
         <link name="${name}">
             <visual>
@@ -34,4 +48,9 @@
                 <origin xyz="${origin_xyz}" rpy="0 0 0"></origin>
             </collision>
+            <inertial>
+                <origin xyz="${origin_xyz}" rpy="0 0 0"></origin>
+                <mass value="${mass}"></mass>
+                <inertia ixx="${ixx}" ixy="0.0" ixz="0.0" iyy="${iyy}" iyz="0.0" izz="${izz}"></inertia>
+            </inertial>
         </link>
     </xacro:macro>

File: tutorial_robots/robot_arm_description/urdf/robot_arm.xacro (robot description, xacro)
@@ -5,4 +5,5 @@
     <xacro:include filename="arm.xacro"></xacro:include>
     <xacro:include filename="gripper.xacro"></xacro:include>
+    <xacro:include filename="object.xacro"></xacro:include>
     <xacro:include filename="robot_arm.ros2_control.xacro"></xacro:include>
     <!-- Fixed joint attaching the gripper base to the tool link -->
@@ -12,3 +13,8 @@
         <origin xyz="0 0 0" rpy="0 0 0"></origin>
     </joint>
+    <joint name="object_joint" type="fixed">
+        <parent link="base_link"></parent>
+        <child link="object"></child>
+        <origin xyz="0 -1.0 0.25" rpy="0 0 0"></origin>
+    </joint>
 </robot>

Commit message: Make robot spawn in Rviz and Gazebo

File: tutorial_robots/robot_arm_description/urdf/arm.xacro (robot description, xacro)
@@ -1,4 +1,5 @@
 <?xml version="1.0"?>
 <robot xmlns:xacro="http://www.ros.org/wiki/xacro">
+    <link name="world"></link>
     <link name="base_footprint"></link>
     <xacro:property name="base_link_length" value="0.5"></xacro:property>
@@ -41,4 +42,10 @@
     </link>
     <!-- Joints -->
+    <!-- Anchor base to world so arm doesn't fall in Gazebo -->
+    <joint name="world_base_footprint_joint" type="fixed">
+        <parent link="world"></parent>
+        <child link="base_footprint"></child>
+        <origin xyz="0 0 0" rpy="0 0 0"></origin>
+    </joint>
     <!-- Virtual joint to connect the robot to the world frame -->
     <joint name="base_footprint_joint" type="fixed">
@@ -46,5 +53,5 @@
         <child link="base_link"></child>
         <origin xyz="0 0 0" rpy="0 0 0"></origin>
-        <dynamics friction="0.5" damping="0.5"/>
+        <dynamics friction="2.0" damping="5.0"/>
     </joint>
     <!-- 1 -->
@@ -55,5 +62,5 @@
         <axis xyz="0 0 1"></axis>
         <limit effort="100.0" velocity="1.0" lower="-3.14" upper="3.14"></limit>
-        <dynamics friction="0.5" damping="0.5"/>
+        <dynamics friction="2.0" damping="5.0"/>
     </joint>
     <!-- 2 -->
@@ -64,5 +71,5 @@
         <axis xyz="0 1 0"></axis>
         <limit effort="100.0" velocity="1.0" lower="0.0" upper="2.5"></limit>
-        <dynamics friction="0.5" damping="0.5"/>
+        <dynamics friction="2.0" damping="5.0"/>
     </joint>
     <!-- 3 -->
@@ -73,5 +80,5 @@
         <axis xyz="0 1 0"></axis>
         <limit effort="100.0" velocity="1.0" lower="0.0" upper="2.5"></limit>
-        <dynamics friction="0.5" damping="0.5"/>
+        <dynamics friction="2.0" damping="5.0"/>
     </joint>
     <!-- 4 -->
@@ -82,5 +89,5 @@
         <axis xyz="0 0 1"></axis>
         <limit effort="100.0" velocity="1.0" lower="-3.14" upper="3.14"></limit>
-        <dynamics friction="0.5" damping="0.5"/>
+        <dynamics friction="2.0" damping="5.0"/>
     </joint>
     <!-- 5 -->
@@ -91,5 +98,5 @@
         <axis xyz="0 1 0"></axis>
         <limit effort="100.0" velocity="1.0" lower="-1.57" upper="1.57"></limit>
-        <dynamics friction="0.5" damping="0.5"/>
+        <dynamics friction="2.0" damping="5.0"/>
     </joint>
     <!-- 6 -->

File: tutorial_robots/robot_arm_description/urdf/links_macro.xacro (robot description, xacro)
@@ -1,5 +1,5 @@
 <?xml version="1.0"?>
 <robot xmlns:xacro="http://www.ros.org/wiki/xacro">
-    <xacro:property name="default_density" value="500.0"></xacro:property>
+    <xacro:property name="default_density" value="5.0"></xacro:property>
     <xacro:macro name="box_link" params="name length width height origin_xyz material">
         <xacro:property name="mass" value="${default_density * length * width * height}"></xacro:property>

File: tutorial_robots/robot_arm_description/urdf/object.xacro (robot description, xacro)
@@ -4,5 +4,5 @@
     <xacro:property name="object_width" value="0.1"></xacro:property>
     <xacro:property name="object_height" value="0.5"></xacro:property>
-    <xacro:property name="object_density" value="500.0"></xacro:property>
+    <xacro:property name="object_density" value="5.0"></xacro:property>
     <xacro:property name="object_mass" value="${object_density * object_length * object_width * object_height}"></xacro:property>
     <xacro:property name="object_ixx" value="${object_mass * (object_width*object_width + object_height*object_height) / 12.0}"></xacro:property>
@@ -11,5 +11,5 @@
     <link name="object">
             <inertial>
-                <origin xyz="0 0 0" rpy="0 0 0"></origin>
+                <origin xyz="0 0 0" rpy="0 0 1.57"></origin>
                 <mass value="${object_mass}"></mass>
                 <inertia ixx="${object_ixx}" ixy="0.0" ixz="0.0" iyy="${object_iyy}" iyz="0.0" izz="${object_izz}"></inertia>

File: tutorial_robots/robot_arm_description/urdf/robot_arm.xacro (robot description, xacro)
@@ -7,4 +7,5 @@
     <xacro:include filename="object.xacro"></xacro:include>
     <xacro:include filename="robot_arm.ros2_control.xacro"></xacro:include>
+    <xacro:include filename="robot_arm_gazebo.xacro"></xacro:include>
     <!-- Fixed joint attaching the gripper base to the tool link -->
     <joint name="tool_gripper_joint" type="fixed">
